Commit message: ⚡️ Sentinel: [HIGH] Fix SQL injection vulnerability in recording library
Co-authored-by: dieterolson <198168927+dieterolson@users.noreply.github.com>

File: src/engines/physics_engines/pinocchio/models/generated/golfer.urdf (robot description, URDF)
Before this commit: robot golfer, 47 links, 46 joints
Links:
- removed link right_grip_attachment
Joints:
- removed joint hand_right_to_right_grip_attachment

File: src/shared/urdf/simple_humanoid.urdf (robot description, URDF)
Before this commit: robot simple_humanoid, 6 links, 5 joints
Links:
- link head: mass 4.86 -> 2
- link left_upper_arm: mass 1.96 -> 1
- link left_upper_leg: mass 7.0 -> 3
- link right_upper_arm: mass 1.96 -> 1
- link right_upper_leg: mass 7.0 -> 3
- link torso: mass 30.42 -> 10
