Commit message: feat(pinocchio): add mid-hands frame + floating base to golfer.urdf (closes #4112)
* Insert virtual `mid_hands` link at the geometric centre of the grip
  (midpoint of `hand_left_tip` and `hand_right_tip` frames in the address
  pose) as a fixed-joint child of `thorax3`.
* Reparent `club_shaft` from `hand_left` to `mid_hands` via the new
  `mid_hands_to_club_shaft` fixed joint, realising the cross-engine
  parity-spec §2.6 requirement that the club is locked to the mid-hands
  frame rather than to a single hand.
* Document `pelvis`-as-root pattern in both URDFs: callers attach the
  6-DOF floating base at load time via `pin.JointModelFreeFlyer()`.
* Header comment blocks declare scope of `golfer.urdf` (forward sim with
  club welded) vs `golfer_ik.urdf` (body-only IK target, club tracked
  externally).
* New tests:
  - `tests/heavy_integration/test_pinocchio_urdf_mid_hands.py` exercises
    the live URDF through pinocchio and asserts `nq=30`, root joint is
    `JointModelFreeFlyer`, `mid_hands` frame is within 1 cm of the
    geometric mean of the hand frames at neutral pose, and that
    `club_shaft` is now offset from `mid_hands` (not `hand_left`).
  - `tests/unit/engines/pinocchio/test_golfer_urdf_invariants.py` is a
    pinocchio-free XML-level guard for the same contracts so CI catches
    regressions even when pinocchio is unavailable.
* Update Pinocchio README with a new "golfer.urdf vs golfer_ik.urdf"
  section and example loader snippet.

Co-Authored-By: Claude Opus 4.7 (1M context) <noreply@anthropic.com>

File: src/engines/physics_engines/pinocchio/models/generated/golfer.urdf (robot description, URDF)
Before this commit: robot golfer, 46 links, 45 joints
Links:
- added link mid_hands, mass 0.001
Joints:
- removed joint hand_left_to_club_shaft
- added joint mid_hands_to_club_shaft: type fixed, parent mid_hands, child club_shaft, origin xyz=0.0 0.0 -0.05 rpy=0.0 0.0 0.0
- added joint thorax3_to_mid_hands: type fixed, parent thorax3, child mid_hands, origin xyz=0.0 0.0 -0.17 rpy=0.0 0.0 0.0
